File: secure-element.sch (KiCad schematic (older format))
At the start: 3 parts, among them U8 ATECC608A-SSHDA

Commit message: Add digikey pn's to schematic, update BOM
Parts:
- C16: Digikey (none) -> 311-1439-1-ND
- C17: Digikey (none) -> 490-14603-1-ND
- U8: Digikey (none) -> ATECC608A-SSHCZ-TCT-ND
Changed lines of the file:
@@
 F 3 "http://ww1.microchip.com/downloads/en/DeviceDoc/ATECC608A-CryptoAuthentication-Device-Summary-Data-Sheet-DS40001977B.pdf" H 5600 4000 50  0001 C CNN
 F 4 "C376619" H 5450 3750 50  0001 C CNN "LCSC"
+F 5 "ATECC608A-SSHCZ-TCT-ND" H 5450 3750 50  0001 C CNN "Digikey"
 	1    5450 3750
 	1    0    0    -1
@@
 F 3 "~" H 4200 3750 50  0001 C CNN
 F 4 "C1525" H 4200 3750 50  0001 C CNN "LCSC"
+F 5 "490-14603-1-ND" H 4200 3750 50  0001 C CNN "Digikey"
 	1    4200 3750
 	1    0    0    -1
@@
 F 3 "~" H 3800 3750 50  0001 C CNN
 F 4 "C52923" H 3800 3750 50  0001 C CNN "LCSC"
+F 5 "311-1439-1-ND" H 3800 3750 50  0001 C CNN "Digikey"
 	1    3800 3750
 	1    0    0    -1
@@
 	5950 3850 5750 3850
 $Comp
-L Graphic:Logo_Open_Hardware_Small #LOGO?
+L Graphic:Logo_Open_Hardware_Small #LOGO5
 U 1 1 5DD38B9F
 P 10750 6900
-F 0 "#LOGO?" H 10750 7175 50  0001 C CNN
+F 0 "#LOGO5" H 10750 7175 50  0001 C CNN
 F 1 "Logo_Open_Hardware_Small" H 10750 6675 50  0001 C CNN
 F 2 "" H 10750 6900 50  0001 C CNN
@@
 $EndComp
 $Comp
-L Graphic:SYM_Radio_Waves_Large #SYM?
+L Graphic:SYM_Radio_Waves_Large #SYM5
 U 1 1 5DD38BA5
 P 10200 6850
-F 0 "#SYM?" H 10200 7050 50  0001 C CNN
+F 0 "#SYM5" H 10200 7050 50  0001 C CNN
 F 1 "SYM_Radio_Waves_Large" H 10200 6600 50  0001 C CNN
 F 2 "" H 10200 6650 50  0001 C CNN

Commit message: PCB REV C0 * Make U8 footprint capable of crypto and fram device * Minor updates to schematic * Minor updates to doc prints * Update bot silk to REV C0
Parts:
- removed U8: ATECC608A-SSHDA, jlcpcb_smt:SOIC-8_3.9x4.9mm_P1.27mm, symbol Security:ATECC608A-SSHDA
- added U8: SOIC8-CRYPTO-FRAM, Package_SO:SOIC-8_3.9x4.9mm_P1.27mm, symbol Custom_KiCAD:SOIC8-CRYPTO-FRAM
Connections:
- net GND: now also U8.1 (A0), U8.2 (A1), U8.3 (A2), U8.4 (GND), U8.7 (WP)
- net I2C_SCL: now also U8.6 (SCL)
- net I2C_SDA: now also U8.5 (SDA)
- net VDD: now also U8.8 (VCC)
Other:
- note added: "NOTE 1"
- note added: "Note 1: U8 can be fitted with either ATECC608A crypto or FM24CL04B FRAM"
Changed lines of the file:
@@
 $EndDescr
-$Comp
-L Security:ATECC608A-SSHDA U8
-U 1 1 5D8DE4B5
-P 5450 3750
-F 0 "U8" H 5100 4050 50  0000 R CNN
-F 1 "ATECC608A-SSHDA" H 5150 3950 50  0000 R CNN
-F 2 "jlcpcb_smt:SOIC-8_3.9x4.9mm_P1.27mm" H 5450 3750 50  0001 C CNN
-F 3 "http://ww1.microchip.com/downloads/en/DeviceDoc/ATECC608A-CryptoAuthentication-Device-Summary-Data-Sheet-DS40001977B.pdf" H 5600 4000 50  0001 C CNN
-F 4 "C376619" H 5450 3750 50  0001 C CNN "LCSC"
-F 5 "ATECC608A-SSHCZ-TCT-ND" H 5450 3750 50  0001 C CNN "Digikey"
-	1    5450 3750
-	1    0    0    -1
-$EndComp
 $Comp
 L Device:C C17
@@
 Connection ~ 4200 4250
 Wire Wire Line
-	4200 4250 5450 4250
-Text HLabel 5950 3650 2    50   BiDi Italic 0
+	4200 4250 4900 4250
+Text HLabel 5950 3750 2    50   BiDi Italic 0
 I2C_SDA
 Text HLabel 5950 3850 2    50   Input Italic 0
 I2C_SCL
-Wire Wire Line
-	5950 3650 5750 3650
 Wire Wire Line
 	5950 3850 5750 3850
@@
 EndData
 $EndBitmap
-Text Notes 7000 6700 0    50   Italic 0
+Text Notes 9850 6650 0    50   Italic 0
 https://www.adafruit.com/feather
 $Bitmap
@@
 EndData
 $EndBitmap
+$Comp
+L Custom_KiCAD:SOIC8-CRYPTO-FRAM U8
+U 1 1 5E0CF6E5
+P 5450 3750
+F 0 "U8" H 5650 4150 50  0000 C CNN
+F 1 "SOIC8-CRYPTO-FRAM" H 6000 4050 50  0000 C CNN
+F 2 "Package_SO:SOIC-8_3.9x4.9mm_P1.27mm" H 5450 3750 50  0001 C CNN
+F 3 "http://ww1.microchip.com/downloads/en/DeviceDoc/ATECC608A-CryptoAuthentication-Device-Summary-Data-Sheet-DS40001977B.pdf" H 5600 4000 50  0001 C CNN
+	1    5450 3750
+	1    0    0    -1
+$EndComp
+Wire Wire Line
+	5950 3750 5750 3750
+Wire Wire Line
+	5750 3650 6500 3650
+Wire Wire Line
+	6500 3650 6500 4250
+Wire Wire Line
+	6500 4250 5450 4250
+Wire Wire Line
+	5150 3650 4900 3650
+Wire Wire Line
+	4900 3650 4900 3750
+Connection ~ 4900 4250
+Wire Wire Line
+	4900 4250 5450 4250
+Wire Wire Line
+	5150 3750 4900 3750
+Connection ~ 4900 3750
+Wire Wire Line
+	4900 3750 4900 3850
+Wire Wire Line
+	5150 3850 4900 3850
+Connection ~ 4900 3850
+Wire Wire Line
+	4900 3850 4900 4250
+Text Notes 5600 3300 0    50   ~ 10
+NOTE 1
+Text Notes 750  6500 0    50   Italic 0
+Note 1:  U8 can be fitted with either ATECC608A crypto or FM24CL04B FRAM
 $EndSCHEMATC
